File: Hardware/motor.kicad_sch (KiCad schematic)
At the start: 27 parts

Commit message: changed 1N4148 JLCPCB code and value of R1 and R00000 resistor.
Parts:
- R00000: LCSC C22775 -> C227664
- R1: LCSC C22775 -> C21190
