File: Hardware/supply.kicad_sch (KiCad schematic)
At the start: 39 parts, among them J11 dG300-5.0-02P-13-00AH, J4 CONN_01x03, J6 CONN_01x09, Q1 BSS138, Q2 BSS138, Q3 BSS138, Q4 BSS138, U1 LMS78_05-2.0R, U7 LD1117DT33TR

Commit message: changed 1N4148 JLCPCB code and value of R1 and R00000 resistor.
Parts:
- D10, D11, D12, D13: LCSC C2128 -> C81598
Changed lines of the file:
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@@
       (effects (font (size 1.27 1.27)) hide)
     )
-    (property "LCSC" "C2128" (id 4) (at 121.92 26.67 0)
+    (property "LCSC" "C81598" (id 4) (at 121.92 26.67 0)
       (effects (font (size 1.27 1.27)) hide)
     )
@@
       (effects (font (size 1.27 1.27)) hide)
     )
-    (property "LCSC" "C2128" (id 4) (at 76.2 26.67 0)
+    (property "LCSC" "C81598" (id 4) (at 76.2 26.67 0)
       (effects (font (size 1.27 1.27)) hide)
     )
@@
       (effects (font (size 1.27 1.27)) hide)
     )
-    (property "LCSC" "C2128" (id 4) (at 167.64 26.67 0)
+    (property "LCSC" "C81598" (id 4) (at 167.64 26.67 0)
       (effects (font (size 1.27 1.27)) hide)
     )
@@
       (effects (font (size 1.27 1.27)) hide)
     )
-    (property "LCSC" "C2128" (id 4) (at 218.44 118.11 0)
-      (effects (font (size 1.27 1.27)) hide)
-    )
+    (property "LCSC" "C81598" (id 4) (at 218.44 118.11 0)
+      (effects (font (size 1.27 1.27)) hide)
+    )
