File: Hardware/RobotMotorController/supply.kicad_sch (KiCad schematic)
At the start: 39 parts, among them J11 dG300-5.0-02P-13-00AH, J4 CONN_01x03, J6 CONN_01x09, Q1 BSS138, Q2 BSS138, Q3 BSS138, Q4 BSS138, U1 LMS78_05-2.0R, U7 LD1117DT33TR

Commit message: ADC init completed
Other:
- note added: "ADC1_IN0"
Changed lines of the file:
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@@
     )
+  )
+  (text "ADC1_IN0" (at 86.36 176.53 0)
+    (effects (font (size 1.27 1.27)) (justify left bottom))
   )
   (label "O_MOT" (at 198.12 38.1 0)

Commit message: General update, first encoder implementation
Parts:
- R15, R16, R33, R34, R35, R36, R37, R38, R39, R40, R41: Spice_Model 1k -> (none); Spice_Netlist_Enabled Y -> (none); Spice_Primitive R -> (none)
