File: Hardware/RobotMotorController/RobotMotorController.kicad_pcb (KiCad board)
At the start: 2 copper layers, 74.2 x 92.7 mm, 186 parts, among them J1 PinSocket_2x16_P2.54mm_Vertic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, J10 CONN_01x04, J11 dG300-5.0-02P-13-00AH, J2 PinSocket_2x24_P2.54mm_Vertic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, J3 PinSocket_2x24_P2.54mm_Vertic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, J4 CONN_01x03, J5 CONN_01x04, J6 CONN_01x09, J7 CONN_01x04, J8 CONN_01x04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

Commit message: Aggiornamento Kicad
Parts:
- moved R00000 4.90 mm to (165.7, 117.4)
